File: docs/hw/eagle/MyEasyPort/MyEasyPort.brd (EAGLE design)
At the start: 100 x 80 mm, 11 parts

Commit message: More report refinements and presentation nonsense
Connections:
- removed net VBUS: JP3.19, U$1.10, U$1.16, U$2.10, U$2.16, U$3.10, U$3.16, U$4.10, U$4.16, U$5.10, U$5.16, U$6.10, U$6.16, U$7.10, U$7.16, U$8.10, U$8.16
- new net 3.3V+: JP3.20, U$1.10, U$1.16, U$2.10, U$2.16, U$3.10, U$3.16, U$4.10, U$4.16, U$5.10, U$5.16, U$6.10, U$6.16, U$7.10, U$7.16, U$8.10, U$8.16
Changed lines of the file:
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@@
 <wire x1="32.385" y1="26.1366" x2="52.705" y2="26.1366" width="0" layer="19" extent="1-1"/>
 </signal>
-<signal name="VBUS">
+<signal name="3.3V+">
 <contactref element="U$1" pad="16"/>
 <contactref element="U$1" pad="10"/>
@@
 <contactref element="U$7" pad="16"/>
 <contactref element="U$8" pad="16"/>
-<contactref element="JP3" pad="19"/>
 <contactref element="U$8" pad="10"/>
 <contactref element="U$7" pad="10"/>
@@
 <contactref element="U$3" pad="10"/>
 <contactref element="U$2" pad="10"/>
+<contactref element="JP3" pad="20"/>
 <wire x1="88.265" y1="52.6034" x2="95.885" y2="52.6034" width="0" layer="19" extent="1-1"/>
 <wire x1="79.375" y1="52.6034" x2="88.265" y2="52.6034" width="0" layer="19" extent="1-1"/>
@@
 <wire x1="40.005" y1="52.6034" x2="52.705" y2="52.6034" width="0" layer="19" extent="1-1"/>
 <wire x1="32.385" y1="52.6034" x2="40.005" y2="52.6034" width="0" layer="19" extent="1-1"/>
-<wire x1="74.93" y1="68.58" x2="71.755" y2="52.6034" width="0" layer="19" extent="1-1"/>
+<wire x1="74.93" y1="71.12" x2="71.755" y2="52.6034" width="0" layer="19" extent="1-1"/>
 <wire x1="95.885" y1="26.1366" x2="95.885" y2="52.6034" width="0" layer="19" extent="1-1"/>
 <wire x1="88.265" y1="26.1366" x2="95.885" y2="26.1366" width="0" layer="19" extent="1-1"/>
