File: docs/hw/eagle/MyEasyPort/MyEasyPort.sch (EAGLE design)
At the start: 11 parts

Commit message: More report refinements and presentation nonsense
Connections:
- removed net VBUS: JP3.19, U$1.EN2, U$1.VDD2, U$2.EN2, U$2.VDD2, U$3.EN2, U$3.VDD2, U$4.EN2, U$4.VDD2, U$5.EN2, U$5.VDD2, U$6.EN2, U$6.VDD2, U$7.EN2, U$7.VDD2, U$8.EN2, U$8.VDD2
- new net 3.3V+: JP3.20, U$1.EN2, U$1.VDD2, U$2.EN2, U$2.VDD2, U$3.EN2, U$3.VDD2, U$4.EN2, U$4.VDD2, U$5.EN2, U$5.VDD2, U$6.EN2, U$6.VDD2, U$7.EN2, U$7.VDD2, U$8.EN2, U$8.VDD2
Changed lines of the file:
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@@
 </segment>
 </net>
-<net name="VBUS" class="0">
+<net name="3.3V+" class="0">
 <segment>
 <pinref part="U$1" gate="G$1" pin="VDD2"/>
@@
 <wire x1="63.5" y1="17.78" x2="63.5" y2="2.54" width="0.1524" layer="91"/>
 <wire x1="63.5" y1="2.54" x2="63.5" y2="-68.58" width="0.1524" layer="91"/>
-<wire x1="63.5" y1="-68.58" x2="167.64" y2="-68.58" width="0.1524" layer="91"/>
-<wire x1="167.64" y1="-68.58" x2="231.14" y2="-68.58" width="0.1524" layer="91"/>
+<wire x1="63.5" y1="-68.58" x2="195.58" y2="-68.58" width="0.1524" layer="91"/>
+<wire x1="195.58" y1="-68.58" x2="231.14" y2="-68.58" width="0.1524" layer="91"/>
 <wire x1="231.14" y1="-68.58" x2="231.14" y2="5.08" width="0.1524" layer="91"/>
 <pinref part="U$1" gate="G$1" pin="EN2"/>
@@
 <pinref part="U$8" gate="G$1" pin="VDD2"/>
 <wire x1="220.98" y1="111.76" x2="231.14" y2="111.76" width="0.1524" layer="91"/>
-<pinref part="JP3" gate="A" pin="19"/>
-<wire x1="177.8" y1="-60.96" x2="167.64" y2="-60.96" width="0.1524" layer="91"/>
-<wire x1="167.64" y1="-60.96" x2="167.64" y2="-68.58" width="0.1524" layer="91"/>
-<junction x="167.64" y="-68.58"/>
-<label x="167.64" y="-60.96" size="1.778" layer="95"/>
 <pinref part="U$8" gate="G$1" pin="EN2"/>
 <wire x1="220.98" y1="96.52" x2="231.14" y2="96.52" width="0.1524" layer="91"/>
@@
 <wire x1="71.12" y1="78.74" x2="63.5" y2="78.74" width="0.1524" layer="91"/>
 <junction x="63.5" y="78.74"/>
+<pinref part="JP3" gate="A" pin="20"/>
+<wire x1="185.42" y1="-60.96" x2="195.58" y2="-60.96" width="0.1524" layer="91"/>
+<wire x1="195.58" y1="-60.96" x2="195.58" y2="-68.58" width="0.1524" layer="91"/>
+<junction x="195.58" y="-68.58"/>
+<label x="190.5" y="-60.96" size="1.778" layer="95"/>
 </segment>
 </net>
